Commit message: R890 修 Gazebo 视觉狗：着色、隐藏白盒载体与近景截图
- 视觉层把 STL 按躯干/髋/大腿/小腿着色，深色狗在白色楼梯上可辨；同时把 model:// 网格 URI 落成 file://。
- lite3_planar 增加 carrier_visual 参数（默认 true）；stairstudy_visual 默认隐藏白盒载体、z-offset 改为 0.04，并透传 payload_dir。
- 官方 stairstudy.launch 的载体与碰撞不变；视觉狗仍 static、无碰撞、不判爬楼。
- 同步替换官网两图：白盒载体图与深色狗近景图；未改判据、calibration 或 #151。

File: ws/src/95_simulation/lite3_gazebo_sim/urdf/lite3_planar.urdf.xacro (robot description, xacro)
@@ -14,4 +14,5 @@
 -->
 <robot name="lite3_planar" xmlns:xacro="http://www.ros.org/wiki/xacro">
+  <xacro:arg name="carrier_visual" default="true"/>
   <xacro:property name="lidar_z" value="0.34"/><xacro:property name="lidar_pitch_deg" value="15"/><!-- ★R409 乙（真人 2026-10-19 两句到签＝★符号＝下倾 15° ‖ ★离地目标＝0.45 m）。本行存★度数与★安装高；★槽位硬约束＝rpy 三元＝(roll, pitch, yaw)＝绕 X,Y,Z，雷达前向＝+X ⇒ 要让光轴俯仰必须把角度放进★第二槽（绕 Y 的 pitch）；★放进第一槽＝把雷达侧倾（★本 boot 首刀就踩过、R409 自纠留名）。rpy 单位是弧度 ⇒ 展开处必须写 ${radians(lidar_pitch_deg)}、★不得把 15 直接填进去（那是 15 弧度）。0.34 的算法＝目标离地 0.45 − ★实测稳态基座 0.11（R405 活体窗），★不是按 spawn 初始位 0.15 推的 0.30＝★坑68 的直接兑现。 -->
   <!-- ================= 官方骨架：TORSO（保持官方名；M2R5 起非 root，恒等挂于 base_link 下） ================= -->
@@ -22,9 +23,11 @@
       <inertia ixx="0.3406" iyy="0.1806" izz="0.2810" ixy="0" ixz="0" iyz="0"/>
     </inertial>
-    <visual>
-      <origin xyz="0 0 0" rpy="0 0 0"/>
-      <geometry><box size="0.42 0.31 0.22"/></geometry>
-      <material name="torso_grey"><color rgba="0.35 0.35 0.4 1"/></material>
-    </visual>
+    <xacro:if value="$(arg carrier_visual)">
+      <visual>
+        <origin xyz="0 0 0" rpy="0 0 0"/>
+        <geometry><box size="0.42 0.31 0.22"/></geometry>
+        <material name="torso_grey"><color rgba="0.35 0.35 0.4 1"/></material>
+      </visual>
+    </xacro:if>
     <collision>
       <origin xyz="0 0 0" rpy="0 0 0"/>
@@ -58,8 +61,10 @@
       <inertia ixx="1e-4" iyy="1e-4" izz="1e-4" ixy="0" ixz="0" iyz="0"/>
     </inertial>
-    <visual>
-      <geometry><cylinder radius="0.045" length="0.03"/></geometry>
-      <material name="lidar_black"><color rgba="0.05 0.05 0.05 1"/></material>
-    </visual>
+    <xacro:if value="$(arg carrier_visual)">
+      <visual>
+        <geometry><cylinder radius="0.045" length="0.03"/></geometry>
+        <material name="lidar_black"><color rgba="0.05 0.05 0.05 1"/></material>
+      </visual>
+    </xacro:if>
     <!-- D-M1-5 取舍声明④：sensor 起点不得落于任何自身 collision 内——collision 整块删除（M1 返工 R1 已收口），仅注释留位 -->
   </link>
